File: PCB/Balancing_cam/IMU.kicad_sch (KiCad schematic)
At the start: 4 parts, among them IC1 ICM-42688-P

Commit message: Started with more stuff tho battery chargeis wip
Other:
- title: (none) -> Balancing_cam
Changed lines of the file:
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@@
 	(generator_version "10.0")
 	(paper "A4")
+	(title_block
+		(title "Balancing_cam")
+	)
 	(junction
 		(at 154.94 101.6)
