File: PCB/Balancing_cam/IMU.kicad_sch (KiCad schematic)
At the start: 6 parts, among them U6 LSM6DS3

Commit message: Done, and completed bom
Parts:
- added TP4, TP5: TestPoint, TestPoint:TestPoint_Pad_D1.5mm, symbol Connector:TestPoint
- C31: renamed from C29; LCSC# (none) -> C14442
- C32: renamed from C30; LCSC# (none) -> C14442
- R13: renamed from R12; LCSC# (none) -> C2906861
- R14: renamed from R13; LCSC# (none) -> C2906861
- R15: renamed from R14; LCSC# (none) -> C2906858
Connections:
- net INT1: now also TP4.1
- net at R15.2, U6.12 (CS): now also TP5.1

Commit message: Fixed Bom and added more GND fill
Parts:
- C31, C32: LCSC# C14442 -> C307331
- TP4, TP5: now left out of the parts list
Changed lines of the file:
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@@
 		(body_style 1)
 		(exclude_from_sim no)
-		(in_bom yes)
+		(in_bom no)
 		(on_board yes)
 		(in_pos_files yes)
@@
 		(body_style 1)
 		(exclude_from_sim no)
-		(in_bom yes)
+		(in_bom no)
 		(on_board yes)
 		(in_pos_files yes)
@@
 			)
 		)
-		(property "LCSC#" "C14442"
+		(property "LCSC#" "C307331"
 			(at 144.78 69.85 0)
 			(hide yes)
@@
 			)
 		)
-		(property "LCSC#" "C14442"
+		(property "LCSC#" "C307331"
 			(at 132.08 69.85 0)
 			(hide yes)
