File: PCB/Balancing_cam/Motor_drivers.kicad_sch (KiCad schematic)
At the start: 10 parts, among them U3 TMC2209-LA

Commit message: Started with more stuff tho battery chargeis wip
Parts:
- added R12: 1k, symbol Device:R
Connections:
- net UART renamed RX
- net RX: now also R12.1
- new net TX: R12.2
Other:
- title: (none) -> Balancing_cam
