File: PCB/Balancing_cam/Motor_drivers.kicad_sch (KiCad schematic)
At the start: 14 parts, among them U1 TMC2209-LA

Commit message: Done, and completed bom
Parts:
- C1, C2, C3, C4, C8, C9: LCSC# (none) -> C14442
- C6: LCSC# (none) -> C57895
- C7: LCSC# (none) -> C84703
- R1, R2: LCSC# (none) -> C309528
Changed lines of the file:
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@@
 		(dnp no)
 		(fields_autoplaced yes)
-		(property "Reference" "#PWR03"
+		(property "Reference" "#PWR06"
 			(at 123.19 64.77 0)
 			(hide yes)
@@
 			(project "Balancing_cam"
 				(path "/4f3cb630-ed40-44c6-96ef-050dfa6679a9/232ccfaa-66e9-445a-8ff7-8fafb59cd86d"
-					(reference "#PWR013")
+					(reference "#PWR016")
 					(unit 1)
 				)
 				(path "/4f3cb630-ed40-44c6-96ef-050dfa6679a9/8a519f58-1cea-4f81-be04-058561b76400"
-					(reference "#PWR03")
+					(reference "#PWR06")
 					(unit 1)
 				)
@@
 			)
 		)
-		(property "LCSC#" ""
+		(property "LCSC#" "C14442"
 			(at 123.19 53.34 0)
 			(hide yes)
@@
 			)
 		)
+		(property "LCSC#" "C14442"
+			(at 162.56 114.3 0)
+			(hide yes)
+			(show_name no)
+			(do_not_autoplace no)
+			(effects
+				(font
+					(size 1.27 1.27)
+				)
+			)
+		)
 		(pin "2"
 		)
@@
 		(dnp no)
 		(fields_autoplaced yes)
-		(property "Reference" "#PWR05"
+		(property "Reference" "#PWR08"
 			(at 105.41 87.63 0)
 			(hide yes)
@@
 			(project "Balancing_cam"
 				(path "/4f3cb630-ed40-44c6-96ef-050dfa6679a9/232ccfaa-66e9-445a-8ff7-8fafb59cd86d"
-					(reference "#PWR015")
+					(reference "#PWR018")
 					(unit 1)
 				)
 				(path "/4f3cb630-ed40-44c6-96ef-050dfa6679a9/8a519f58-1cea-4f81-be04-058561b76400"
-					(reference "#PWR05")
+					(reference "#PWR08")
 					(unit 1)
 				)
@@
 			)
 		)
-		(property "LCSC#" ""
+		(property "LCSC#" "C14442"
 			(at 134.62 53.34 0)
 			(hide yes)
@@
 			)
 		)
-		(property "LCSC#" ""
+		(property "LCSC#" "C309528"
 			(at 176.53 109.22 90)
 			(hide yes)
@@
 		(dnp no)
 		(fields_autoplaced yes)
-		(property "Reference" "#PWR06"
+		(property "Reference" "#PWR09"
 			(at 166.37 87.63 0)
 			(hide yes)
@@
 			(project "Balancing_cam"
 				(path "/4f3cb630-ed40-44c6-96ef-050dfa6679a9/232ccfaa-66e9-445a-8ff7-8fafb59cd86d"
-					(reference "#PWR016")
+					(reference "#PWR019")
 					(unit 1)
 				)
 				(path "/4f3cb630-ed40-44c6-96ef-050dfa6679a9/8a519f58-1cea-4f81-be04-058561b76400"
-					(reference "#PWR06")
+					(reference "#PWR09")
 					(unit 1)
 				)
@@
 		(dnp no)
 		(fields_autoplaced yes)
-		(property "Reference" "#PWR09"
+		(property "Reference" "#PWR012"
 			(at 156.21 127 0)
 			(hide yes)
@@
 			(project "Balancing_cam"
 				(path "/4f3cb630-ed40-44c6-96ef-050dfa6679a9/232ccfaa-66e9-445a-8ff7-8fafb59cd86d"
-					(reference "#PWR019")
+					(reference "#PWR022")
 					(unit 1)
 				)
 				(path "/4f3cb630-ed40-44c6-96ef-050dfa6679a9/8a519f58-1cea-4f81-be04-058561b76400"
-					(reference "#PWR09")
+					(reference "#PWR012")
 					(unit 1)
 				)
@@
 		(dnp no)
 		(fields_autoplaced yes)
-		(property "Reference" "#PWR07"
+		(property "Reference" "#PWR010"
 			(at 184.15 116.84 0)
 			(hide yes)
@@
 			(project "Balancing_cam"
 				(path "/4f3cb630-ed40-44c6-96ef-050dfa6679a9/232ccfaa-66e9-445a-8ff7-8fafb59cd86d"
-					(reference "#PWR017")
+					(reference "#PWR020")
 					(unit 1)
 				)
 				(path "/4f3cb630-ed40-44c6-96ef-050dfa6679a9/8a519f58-1cea-4f81-be04-058561b76400"
-					(reference "#PWR07")
+					(reference "#PWR010")
 					(unit 1)
 				)
@@
 		(dnp no)
 		(fields_autoplaced yes)
-		(property "Reference" "#PWR02"
+		(property "Reference" "#PWR05"
 			(at 161.29 50.8 0)
 			(hide yes)
@@
 			(project "Balancing_cam"
 				(path "/4f3cb630-ed40-44c6-96ef-050dfa6679a9/232ccfaa-66e9-445a-8ff7-8fafb59cd86d"
-					(reference "#PWR012")
+					(reference "#PWR015")
 					(unit 1)
 				)
 				(path "/4f3cb630-ed40-44c6-96ef-050dfa6679a9/8a519f58-1cea-4f81-be04-058561b76400"
-					(reference "#PWR02")
+					(reference "#PWR05")
 					(unit 1)
 				)
@@
 			)
 		)
+		(property "LCSC#" "C14442"
+			(at 149.86 114.3 0)
+			(hide yes)
+			(show_name no)
+			(do_not_autoplace no)
+			(effects
+				(font
+					(size 1.27 1.27)
+				)
+			)
+		)
 		(pin "2"
 		)
@@
 		(dnp no)
 		(fields_autoplaced yes)
-		(property "Reference" "#PWR010"
+		(property "Reference" "#PWR013"
 			(at 68.58 139.7 0)
 			(hide yes)
@@
 			(project "Balancing_cam"
 				(path "/4f3cb630-ed40-44c6-96ef-050dfa6679a9/232ccfaa-66e9-445a-8ff7-8fafb59cd86d"
-					(reference "#PWR020")
+					(reference "#PWR023")
 					(unit 1)
 				)
 				(path "/4f3cb630-ed40-44c6-96ef-050dfa6679a9/8a519f58-1cea-4f81-be04-058561b76400"
-					(reference "#PWR010")
+					(reference "#PWR013")
 					(unit 1)
 				)
@@
 			)
 		)
-		(property "LCSC#" ""
+		(property "LCSC#" "C14442"
 			(at 147.32 53.34 0)
 			(hide yes)
@@
 			)
 		)
-		(property "LCSC#" ""
+		(property "LCSC#" "C84703"
 			(at 154.94 83.82 0)
 			(hide yes)
@@
 		(dnp no)
 		(fields_autoplaced yes)
-		(property "Reference" "#PWR08"
+		(property "Reference" "#PWR011"
 			(at 130.81 125.73 0)
 			(hide yes)
@@
 			(project "Balancing_cam"
 				(path "/4f3cb630-ed40-44c6-96ef-050dfa6679a9/232ccfaa-66e9-445a-8ff7-8fafb59cd86d"
-					(reference "#PWR018")
+					(reference "#PWR021")
 					(unit 1)
 				)
 				(path "/4f3cb630-ed40-44c6-96ef-050dfa6679a9/8a519f58-1cea-4f81-be04-058561b76400"
-					(reference "#PWR08")
+					(reference "#PWR011")
 					(unit 1)
 				)
@@
 			)
 		)
-		(property "LCSC#" ""
+		(property "LCSC#" "C309528"
 			(at 176.53 106.68 90)
 			(hide yes)
@@
 		(dnp no)
 		(fields_autoplaced yes)
-		(property "Reference" "#PWR04"
+		(property "Reference" "#PWR07"
 			(at 161.29 66.04 0)
 			(hide yes)
@@
 			(project "Balancing_cam"
 				(path "/4f3cb630-ed40-44c6-96ef-050dfa6679a9/232ccfaa-66e9-445a-8ff7-8fafb59cd86d"
-					(reference "#PWR014")
+					(reference "#PWR017")
 					(unit 1)
 				)
 				(path "/4f3cb630-ed40-44c6-96ef-050dfa6679a9/8a519f58-1cea-4f81-be04-058561b76400"
-					(reference "#PWR04")
+					(reference "#PWR07")
 					(unit 1)
 				)
@@
 		(dnp no)
 		(fields_autoplaced yes)
-		(property "Reference" "#PWR01"
+		(property "Reference" "#PWR04"
 			(at 119.38 50.8 0)
 			(hide yes)
@@
 			(project "Balancing_cam"
 				(path "/4f3cb630-ed40-44c6-96ef-050dfa6679a9/232ccfaa-66e9-445a-8ff7-8fafb59cd86d"
-					(reference "#PWR011")
+					(reference "#PWR014")
 					(unit 1)
 				)
 				(path "/4f3cb630-ed40-44c6-96ef-050dfa6679a9/8a519f58-1cea-4f81-be04-058561b76400"
-					(reference "#PWR01")
+					(reference "#PWR04")
 					(unit 1)
 				)
@@
 			)
 		)
-		(property "LCSC#" ""
+		(property "LCSC#" "C14442"
 			(at 140.97 53.34 0)
 			(hide yes)
@@
 			)
 		)
-		(property "LCSC#" ""
+		(property "LCSC#" "C57895"
 			(at 166.37 76.2 0)
 			(hide yes)

Commit message: Fixed Bom and added more GND fill
Parts:
- C1, C2, C3, C4, C8, C9: LCSC# C14442 -> C307331
- C7: LCSC# C84703 -> C337699
Changed lines of the file:
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@@
 			)
 		)
-		(property "LCSC#" "C14442"
+		(property "LCSC#" "C307331"
 			(at 123.19 53.34 0)
 			(hide yes)
@@
 			)
 		)
-		(property "LCSC#" "C14442"
+		(property "LCSC#" "C307331"
 			(at 162.56 114.3 0)
 			(hide yes)
@@
 			)
 		)
-		(property "LCSC#" "C14442"
+		(property "LCSC#" "C307331"
 			(at 134.62 53.34 0)
 			(hide yes)
@@
 			)
 		)
-		(property "LCSC#" "C14442"
+		(property "LCSC#" "C307331"
 			(at 149.86 114.3 0)
 			(hide yes)
@@
 			)
 		)
-		(property "LCSC#" "C14442"
+		(property "LCSC#" "C307331"
 			(at 147.32 53.34 0)
 			(hide yes)
@@
 			)
 		)
-		(property "LCSC#" "C84703"
+		(property "LCSC#" "C337699"
 			(at 154.94 83.82 0)
 			(hide yes)
@@
 			)
 		)
-		(property "LCSC#" "C14442"
+		(property "LCSC#" "C307331"
 			(at 140.97 53.34 0)
 			(hide yes)
