File: PCB/Balancing_cam/Balancing_cam.kicad_sch (KiCad schematic)
At the start: 0 parts

Commit message: Started with more stuff tho battery chargeis wip
Other:
- title: (none) -> Balancing_cam
Changed lines of the file:
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@@
 	(generator_version "10.0")
 	(paper "A4")
+	(title_block
+		(title "Balancing_cam")
+	)
 	(bus
 		(pts

Commit message: Finalized schematic and pcb
Parts:
- added H1, H2, H3: MountingHole_Pad, MountingHole:MountingHole_3.2mm_M3_Pad, symbol Mechanical:MountingHole_Pad
Connections:
- new net GND: H1.1, H2.1, H3.1
Other:
- added sheet Breakout (Breakout.kicad_sch)
- added sheet Motor_connector_1 (Motor_connector.kicad_sch)
- added sheet Motor_connector_2 (Motor_connector.kicad_sch)
- sheet IMU ports: added INT1; removed INT
- sheet Microcontroller ports: added CTRL{UART}, IO21, IO36, VTX{UART}, {USB}; removed none
- sheet Motor_1 ports: added none; removed {ADDR}
- sheet Motor_2 ports: added none; removed {ADDR}
- sheet Power_in ports: added FAN, {USB}; removed none
