File: PCB/Balancing_cam/Breakout.kicad_sch (KiCad schematic)
At the start: 11 parts, among them J8 Conn_01x03, J9 Conn_01x04

Commit message: Done, and completed bom
Parts:
- J8: LCSC# (none) -> C160389
- J9: LCSC# (none) -> C7501262
- R22: renamed from R21; LCSC# (none) -> C105588
- R23: renamed from R22; LCSC# (none) -> C105588
- R24: renamed from R23; LCSC# (none) -> C105588
- R25: renamed from R24; LCSC# (none) -> C105588
- renumbered L13 to L14
Changed lines of the file:
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@@
 		(dnp no)
 		(fields_autoplaced yes)
-		(property "Reference" "#PWR080"
+		(property "Reference" "#PWR087"
 			(at 152.4 86.36 0)
 			(hide yes)
@@
 			(project "Balancing_cam"
 				(path "/4f3cb630-ed40-44c6-96ef-050dfa6679a9/b3bf285e-173c-4276-ac97-f19448f9ab02"
-					(reference "#PWR080")
+					(reference "#PWR087")
 					(unit 1)
 				)
@@
 			)
 		)
+		(property "LCSC#" "C7501262"
+			(at 158.75 124.46 0)
+			(hide yes)
+			(show_name no)
+			(do_not_autoplace no)
+			(effects
+				(font
+					(size 1.27 1.27)
+				)
+			)
+		)
 		(pin "3"
 		)
@@
 		(dnp no)
 		(fields_autoplaced yes)
-		(property "Reference" "#PWR086"
+		(property "Reference" "#PWR094"
 			(at 152.4 137.16 0)
 			(hide yes)
@@
 			(project "Balancing_cam"
 				(path "/4f3cb630-ed40-44c6-96ef-050dfa6679a9/b3bf285e-173c-4276-ac97-f19448f9ab02"
-					(reference "#PWR086")
+					(reference "#PWR094")
 					(unit 1)
 				)
@@
 		(dnp no)
 		(fields_autoplaced yes)
-		(property "Reference" "R21"
+		(property "Reference" "R22"
 			(at 146.05 67.31 90)
 			(show_name no)
@@
 		)
 		(property "Mouser Price/Stock" ""
+			(at 146.05 73.66 90)
+			(hide yes)
+			(show_name no)
+			(do_not_autoplace no)
+			(effects
+				(font
+					(size 1.27 1.27)
+				)
+			)
+		)
+		(property "LCSC#" "C105588"
 			(at 146.05 73.66 90)
 			(hide yes)
@@
 			(project "Balancing_cam"
 				(path "/4f3cb630-ed40-44c6-96ef-050dfa6679a9/b3bf285e-173c-4276-ac97-f19448f9ab02"
-					(reference "R21")
+					(reference "R22")
 					(unit 1)
 				)
@@
 		(dnp no)
 		(fields_autoplaced yes)
-		(property "Reference" "#PWR094"
+		(property "Reference" "#PWR088"
 			(at 158.75 91.44 0)
 			(hide yes)
@@
 			(project "Balancing_cam"
 				(path "/4f3cb630-ed40-44c6-96ef-050dfa6679a9/b3bf285e-173c-4276-ac97-f19448f9ab02"
-					(reference "#PWR094")
+					(reference "#PWR088")
 					(unit 1)
 				)
@@
 		(dnp no)
 		(fields_autoplaced yes)
-		(property "Reference" "#PWR078"
+		(property "Reference" "#PWR085"
 			(at 120.65 69.85 0)
 			(hide yes)
@@
 			(project "Balancing_cam"
 				(path "/4f3cb630-ed40-44c6-96ef-050dfa6679a9/b3bf285e-173c-4276-ac97-f19448f9ab02"
-					(reference "#PWR078")
+					(reference "#PWR085")
 					(unit 1)
 				)
@@
 		(dnp no)
 		(fields_autoplaced yes)
-		(property "Reference" "#PWR083"
+		(property "Reference" "#PWR091"
 			(at 125.73 120.65 0)
 			(hide yes)
@@
 			(project "Balancing_cam"
 				(path "/4f3cb630-ed40-44c6-96ef-050dfa6679a9/b3bf285e-173c-4276-ac97-f19448f9ab02"
-					(reference "#PWR083")
+					(reference "#PWR091")
 					(unit 1)
 				)
@@
 		(dnp no)
 		(fields_autoplaced yes)
-		(property "Reference" "#PWR079"
+		(property "Reference" "#PWR086"
 			(at 132.08 69.85 0)
 			(hide yes)
@@
 			(project "Balancing_cam"
 				(path "/4f3cb630-ed40-44c6-96ef-050dfa6679a9/b3bf285e-173c-4276-ac97-f19448f9ab02"
-					(reference "#PWR079")
+					(reference "#PWR086")
 					(unit 1)
 				)
@@
 		(dnp no)
 		(fields_autoplaced yes)
-		(property "Reference" "#PWR082"
+		(property "Reference" "#PWR090"
 			(at 137.16 100.33 0)
 			(hide yes)
@@
 			(project "Balancing_cam"
 				(path "/4f3cb630-ed40-44c6-96ef-050dfa6679a9/b3bf285e-173c-4276-ac97-f19448f9ab02"
-					(reference "#PWR082")
+					(reference "#PWR090")
 					(unit 1)
 				)
@@
 		(in_pos_files yes)
 		(dnp no)
-		(property "Reference" "R22"
+		(property "Reference" "R23"
 			(at 146.0908 82.55 90)
 			(show_name no)
@@
 		)
 		(property "Mouser Price/Stock" ""
+			(at 146.0908 76.2 90)
+			(hide yes)
+			(show_name no)
+			(do_not_autoplace no)
+			(effects
+				(font
+					(size 1.27 1.27)
+				)
+			)
+		)
+		(property "LCSC#" "C105588"
 			(at 146.0908 76.2 90)
 			(hide yes)
@@
 			(project "Balancing_cam"
 				(path "/4f3cb630-ed40-44c6-96ef-050dfa6679a9/b3bf285e-173c-4276-ac97-f19448f9ab02"
-					(reference "R22")
+					(reference "R23")
 					(unit 1)
 				)
@@
 			)
 		)
+		(property "LCSC#" "C160389"
+			(at 158.75 76.2 0)
+			(hide yes)
+			(show_name no)
+			(do_not_autoplace no)
+			(effects
+				(font
+					(size 1.27 1.27)
+				)
+			)
+		)
 		(pin "3"
 		)
@@
 		(dnp no)
 		(fields_autoplaced yes)
-		(property "Reference" "R23"
+		(property "Reference" "R24"
 			(at 148.59 115.57 90)
 			(show_name no)
@@
 		)
 		(property "Mouser Price/Stock" ""
+			(at 148.59 121.92 90)
+			(hide yes)
+			(show_name no)
+			(do_not_autoplace no)
+			(effects
+				(font
+					(size 1.27 1.27)
+				)
+			)
+		)
+		(property "LCSC#" "C105588"
 			(at 148.59 121.92 90)
 			(hide yes)
@@
 			(project "Balancing_cam"
 				(path "/4f3cb630-ed40-44c6-96ef-050dfa6679a9/b3bf285e-173c-4276-ac97-f19448f9ab02"
-					(reference "R23")
+					(reference "R24")
 					(unit 1)
 				)
@@
 		(dnp no)
 		(fields_autoplaced yes)
-		(property "Reference" "#PWR084"
+		(property "Reference" "#PWR092"
 			(at 137.16 120.65 0)
 			(hide yes)
@@
 			(project "Balancing_cam"
 				(path "/4f3cb630-ed40-44c6-96ef-050dfa6679a9/b3bf285e-173c-4276-ac97-f19448f9ab02"
-					(reference "#PWR084")
+					(reference "#PWR092")
 					(unit 1)
 				)
@@
 		(dnp no)
 		(fields_autoplaced yes)
-		(property "Reference" "#PWR076"
+		(property "Reference" "#PWR083"
 			(at 120.65 49.53 0)
 			(hide yes)
@@
 			(project "Balancing_cam"
 				(path "/4f3cb630-ed40-44c6-96ef-050dfa6679a9/b3bf285e-173c-4276-ac97-f19448f9ab02"
-					(reference "#PWR076")
+					(reference "#PWR083")
 					(unit 1)
 				)
@@
 		(dnp no)
 		(fields_autoplaced yes)
-		(property "Reference" "#PWR085"
+		(property "Reference" "#PWR093"
 			(at 100.33 129.54 0)
 			(hide yes)
@@
 			(project "Balancing_cam"
 				(path "/4f3cb630-ed40-44c6-96ef-050dfa6679a9/b3bf285e-173c-4276-ac97-f19448f9ab02"
-					(reference "#PWR085")
+					(reference "#PWR093")
 					(unit 1)
 				)
@@
 		(in_pos_files yes)
 		(dnp no)
-		(property "Reference" "R24"
+		(property "Reference" "R25"
 			(at 148.59 130.81 90)
 			(show_name no)
@@
 		)
 		(property "Mouser Price/Stock" ""
+			(at 148.59 124.46 90)
+			(hide yes)
+			(show_name no)
+			(do_not_autoplace no)
+			(effects
+				(font
+					(size 1.27 1.27)
+				)
+			)
+		)
+		(property "LCSC#" "C105588"
 			(at 148.59 124.46 90)
 			(hide yes)
@@
 			(project "Balancing_cam"
 				(path "/4f3cb630-ed40-44c6-96ef-050dfa6679a9/b3bf285e-173c-4276-ac97-f19448f9ab02"
-					(reference "R24")
+					(reference "R25")
 					(unit 1)
 				)
@@
 		(in_pos_files yes)
 		(dnp no)
-		(property "Reference" "L13"
+		(property "Reference" "L14"
 			(at 110.49 123.952 90)
 			(show_name no)
@@
 			(project "Balancing_cam"
 				(path "/4f3cb630-ed40-44c6-96ef-050dfa6679a9/b3bf285e-173c-4276-ac97-f19448f9ab02"
-					(reference "L13")
+					(reference "L14")
 					(unit 1)
 				)
@@
 		(dnp no)
 		(fields_autoplaced yes)
-		(property "Reference" "#PWR081"
+		(property "Reference" "#PWR089"
 			(at 125.73 100.33 0)
 			(hide yes)
@@
 			(project "Balancing_cam"
 				(path "/4f3cb630-ed40-44c6-96ef-050dfa6679a9/b3bf285e-173c-4276-ac97-f19448f9ab02"
-					(reference "#PWR081")
+					(reference "#PWR089")
 					(unit 1)
 				)
@@
 		(dnp no)
 		(fields_autoplaced yes)
-		(property "Reference" "#PWR077"
+		(property "Reference" "#PWR084"
 			(at 132.08 49.53 0)
 			(hide yes)
@@
 			(project "Balancing_cam"
 				(path "/4f3cb630-ed40-44c6-96ef-050dfa6679a9/b3bf285e-173c-4276-ac97-f19448f9ab02"
-					(reference "#PWR077")
+					(reference "#PWR084")
 					(unit 1)
 				)
