File: PCB/Balancing_cam/Motor_connector.kicad_sch (KiCad schematic)
At the start: 6 parts, among them U6 LSM6DS3

Commit message: Finalized schematic and pcb
Parts:
- removed C29, C30: 100n, Capacitor_SMD:C_0402_1005Metric, symbol Device:C
- removed R12, R13: 10k, Resistor_SMD:R_0402_1005Metric, symbol Device:R
- removed R14: 0R, Resistor_SMD:R_0402_1005Metric, symbol Device:R
- removed U6: LSM6DS3, Package_LGA:LGA-14_3x2.5mm_P0.5mm_LayoutBorder3x4y, symbol Sensor_Motion:LSM6DS3
- added C37, C38, C39, C40: 1n, Capacitor_SMD:C_0603_1608Metric, symbol Device:C
- added J6: Conn_01x04, Connector_JST:JST_XH_B4B-XH-A_1x04_P2.50mm_Vertical, symbol Connector_Generic:Conn_01x04
- added L5, L6, L7, L8: BLM18KG121TN1D, Inductor_SMD:L_0603_1608Metric, symbol Device:L
Connections:
- net GND: now also C37.2, C38.2, C39.2, C40.2
- new net: C38.1, J6.3 (Pin_3), L7.2
- new net: C39.1, J6.2 (Pin_2), L6.2
- new net: C40.1, J6.1 (Pin_1), L5.2
- new net: C37.1, J6.4 (Pin_4), L8.2
- new net OA1: L6.1
- new net OA2: L5.1
- new net OB1: L7.1
- new net OB2: L8.1
- no-connect marks 4 -> 0
Other:
- title: Balancing_cam -> (none)

Commit message: Done, and completed bom
Parts:
- C39: renamed from C37; LCSC# (none) -> C153291
- C40: renamed from C38; LCSC# (none) -> C153291
- C41: renamed from C39; LCSC# (none) -> C153291
- C42: renamed from C40; LCSC# (none) -> C153291
- renumbered L5 to L6, L6 to L7, L7 to L8, L8 to L9
Changed lines of the file:
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@@
 		(in_pos_files yes)
 		(dnp no)
-		(property "Reference" "C38"
+		(property "Reference" "C40"
 			(at 164.846 100.33 0)
 			(show_name no)
@@
 		)
 		(property "Mouser Price/Stock" ""
+			(at 162.56 101.6 0)
+			(hide yes)
+			(show_name no)
+			(do_not_autoplace no)
+			(effects
+				(font
+					(size 1.27 1.27)
+				)
+			)
+		)
+		(property "LCSC#" "C153291"
 			(at 162.56 101.6 0)
 			(hide yes)
@@
 			(project "Balancing_cam"
 				(path "/4f3cb630-ed40-44c6-96ef-050dfa6679a9/ebe462b6-6f01-4c38-9a76-d3bc641349bd"
-					(reference "C38")
+					(reference "C40")
 					(unit 1)
 				)
 				(path "/4f3cb630-ed40-44c6-96ef-050dfa6679a9/f1f331c8-08f7-43f5-94be-a907a264cb62"
-					(reference "C42")
+					(reference "C44")
 					(unit 1)
 				)
@@
 		(in_pos_files yes)
 		(dnp no)
-		(property "Reference" "C39"
+		(property "Reference" "C41"
 			(at 173.736 100.33 0)
 			(show_name no)
@@
 		)
 		(property "Mouser Price/Stock" ""
+			(at 171.45 101.6 0)
+			(hide yes)
+			(show_name no)
+			(do_not_autoplace no)
+			(effects
+				(font
+					(size 1.27 1.27)
+				)
+			)
+		)
+		(property "LCSC#" "C153291"
 			(at 171.45 101.6 0)
 			(hide yes)
@@
 			(project "Balancing_cam"
 				(path "/4f3cb630-ed40-44c6-96ef-050dfa6679a9/ebe462b6-6f01-4c38-9a76-d3bc641349bd"
-					(reference "C39")
+					(reference "C41")
 					(unit 1)
 				)
 				(path "/4f3cb630-ed40-44c6-96ef-050dfa6679a9/f1f331c8-08f7-43f5-94be-a907a264cb62"
-					(reference "C43")
+					(reference "C45")
 					(unit 1)
 				)
@@
 		(in_pos_files yes)
 		(dnp no)
-		(property "Reference" "L5"
+		(property "Reference" "L6"
 			(at 138.43 82.042 90)
 			(show_name no)
@@
 			(project "Balancing_cam"
 				(path "/4f3cb630-ed40-44c6-96ef-050dfa6679a9/ebe462b6-6f01-4c38-9a76-d3bc641349bd"
-					(reference "L5")
+					(reference "L6")
 					(unit 1)
 				)
 				(path "/4f3cb630-ed40-44c6-96ef-050dfa6679a9/f1f331c8-08f7-43f5-94be-a907a264cb62"
-					(reference "L9")
+					(reference "L10")
 					(unit 1)
 				)
@@
 		(in_pos_files yes)
 		(dnp no)
-		(property "Reference" "C37"
+		(property "Reference" "C39"
 			(at 155.956 100.33 0)
 			(show_name no)
@@
 		)
 		(property "Mouser Price/Stock" ""
+			(at 153.67 101.6 0)
+			(hide yes)
+			(show_name no)
+			(do_not_autoplace no)
+			(effects
+				(font
+					(size 1.27 1.27)
+				)
+			)
+		)
+		(property "LCSC#" "C153291"
 			(at 153.67 101.6 0)
 			(hide yes)
@@
 			(project "Balancing_cam"
 				(path "/4f3cb630-ed40-44c6-96ef-050dfa6679a9/ebe462b6-6f01-4c38-9a76-d3bc641349bd"
-					(reference "C37")
+					(reference "C39")
 					(unit 1)
 				)
 				(path "/4f3cb630-ed40-44c6-96ef-050dfa6679a9/f1f331c8-08f7-43f5-94be-a907a264cb62"
-					(reference "C41")
+					(reference "C43")
 					(unit 1)
 				)
@@
 		(in_pos_files yes)
 		(dnp no)
-		(property "Reference" "C40"
+		(property "Reference" "C42"
 			(at 182.626 100.33 0)
 			(show_name no)
@@
 		)
 		(property "Mouser Price/Stock" ""
+			(at 180.34 101.6 0)
+			(hide yes)
+			(show_name no)
+			(do_not_autoplace no)
+			(effects
+				(font
+					(size 1.27 1.27)
+				)
+			)
+		)
+		(property "LCSC#" "C153291"
 			(at 180.34 101.6 0)
 			(hide yes)
@@
 			(project "Balancing_cam"
 				(path "/4f3cb630-ed40-44c6-96ef-050dfa6679a9/ebe462b6-6f01-4c38-9a76-d3bc641349bd"
-					(reference "C40")
+					(reference "C42")
 					(unit 1)
 				)
 				(path "/4f3cb630-ed40-44c6-96ef-050dfa6679a9/f1f331c8-08f7-43f5-94be-a907a264cb62"
-					(reference "C44")
+					(reference "C46")
 					(unit 1)
 				)
@@
 		(dnp no)
 		(fields_autoplaced yes)
-		(property "Reference" "#PWR074"
+		(property "Reference" "#PWR081"
 			(at 181.61 114.3 0)
 			(hide yes)
@@
 			(project "Balancing_cam"
 				(path "/4f3cb630-ed40-44c6-96ef-050dfa6679a9/ebe462b6-6f01-4c38-9a76-d3bc641349bd"
-					(reference "#PWR074")
+					(reference "#PWR081")
 					(unit 1)
 				)
 				(path "/4f3cb630-ed40-44c6-96ef-050dfa6679a9/f1f331c8-08f7-43f5-94be-a907a264cb62"
-					(reference "#PWR075")
+					(reference "#PWR082")
 					(unit 1)
 				)
@@
 		(in_pos_files yes)
 		(dnp no)
-		(property "Reference" "L7"
+		(property "Reference" "L8"
 			(at 138.43 92.202 90)
 			(show_name no)
@@
 			(project "Balancing_cam"
 				(path "/4f3cb630-ed40-44c6-96ef-050dfa6679a9/ebe462b6-6f01-4c38-9a76-d3bc641349bd"
-					(reference "L7")
+					(reference "L8")
 					(unit 1)
 				)
 				(path "/4f3cb630-ed40-44c6-96ef-050dfa6679a9/f1f331c8-08f7-43f5-94be-a907a264cb62"
-					(reference "L11")
+					(reference "L12")
 					(unit 1)
 				)
@@
 		(in_pos_files yes)
 		(dnp no)
-		(property "Reference" "L8"
+		(property "Reference" "L9"
 			(at 138.43 97.282 90)
 			(show_name no)
@@
 			(project "Balancing_cam"
 				(path "/4f3cb630-ed40-44c6-96ef-050dfa6679a9/ebe462b6-6f01-4c38-9a76-d3bc641349bd"
-					(reference "L8")
+					(reference "L9")
 					(unit 1)
 				)
 				(path "/4f3cb630-ed40-44c6-96ef-050dfa6679a9/f1f331c8-08f7-43f5-94be-a907a264cb62"
-					(reference "L12")
+					(reference "L13")
 					(unit 1)
 				)
@@
 		(in_pos_files yes)
 		(dnp no)
-		(property "Reference" "L6"
+		(property "Reference" "L7"
 			(at 138.43 87.122 90)
 			(show_name no)
@@
 			(project "Balancing_cam"
 				(path "/4f3cb630-ed40-44c6-96ef-050dfa6679a9/ebe462b6-6f01-4c38-9a76-d3bc641349bd"
-					(reference "L6")
+					(reference "L7")
 					(unit 1)
 				)
 				(path "/4f3cb630-ed40-44c6-96ef-050dfa6679a9/f1f331c8-08f7-43f5-94be-a907a264cb62"
-					(reference "L10")
-					(unit 1)
-				)
+					(reference "L11")
+					(unit 1)
+				)
