File: PCB/Balancing_cam/Microcontroller.kicad_sch (KiCad schematic)
At the start: 15 parts, among them J1 USB_C_Receptacle_USB2.0_16P, J3 Conn_01x04, SW1 EN, SW2 BOOT, U2 ESP32-S3-MINI-1

Commit message: Started with more stuff tho battery chargeis wip
Parts:
- removed D1: D, symbol Device:D
- removed J1: USB_C_Receptacle_USB2.0_16P, symbol Connector:USB_C_Receptacle_USB2.0_16P
- removed R4, R5: 5.1k, symbol Device:R
Connections:
- no-connect marks 2 -> 0
Other:
- title: (none) -> Balancing_cam

Commit message: Finalized schematic and pcb
Parts:
- added C35, C36: 100n, Capacitor_SMD:C_0402_1005Metric, symbol Device:C
- added D2, D3: BAV99W, Package_TO_SOT_SMD:SOT-23, symbol Diode:BAS40-04
- added D4, D5: WS2812B-4020, footprints:WS2812B-4020, symbol symbols:WS2812B-4020
- added L4: BLM18KG121TN1D, Inductor_SMD:L_0603_1608Metric, symbol Device:L
- added R15, R16: 100R, Resistor_SMD:R_0603_1608Metric, symbol Device:R
- added R20: 1k, Resistor_SMD:R_0402_1005Metric, symbol Device:R
- C31: renamed from C1; footprint (none) -> Capacitor_SMD:C_0603_1608Metric; LCSC# (none) -> C59461
- C32: renamed from C2; footprint (none) -> Capacitor_SMD:C_0402_1005Metric
- C33: renamed from C4; footprint (none) -> Capacitor_SMD:C_0402_1005Metric
- C34: renamed from C3; footprint (none) -> Capacitor_SMD:C_0402_1005Metric
- J5: renamed from J3; footprint (none) -> Connector_PinHeader_2.54mm:PinHeader_1x04_P2.54mm_Vertical
- R17: renamed from R1; footprint (none) -> Resistor_SMD:R_0402_1005Metric
- R18: renamed from R2; footprint (none) -> Resistor_SMD:R_0402_1005Metric
- R19: renamed from R3; footprint (none) -> Resistor_SMD:R_0402_1005Metric
- SW2: renamed from SW1; footprint (none) -> Button_Switch_SMD:SW_SPST_B3U-1000P; LCSC# (none) -> C231329
- SW3: renamed from SW2; footprint (none) -> Button_Switch_SMD:SW_SPST_B3U-1000P; LCSC# (none) -> C231329
- U7: renamed from U2; LCSC# (none) -> C2913206
Connections:
- net GND: now also C35.2, C36.2, D2.1, D3.1, D4.4 (VSS), D5.4 (VSS)
- net IMU.SCL: now also U7.34 (IO38)
- net IMU.SDA: now also U7.33 (IO37)
- net MOT_1.DIAG: now also U7.28 (IO33)
- net MOT_1.DIR: now also U7.14 (IO10)
- net MOT_1.INDEX: now also U7.27 (IO47)
- net MOT_1.STEP: now also U7.15 (IO11)
- net MOT_2.DIAG: now also U7.19 (IO15)
- net MOT_2.DIR: now also U7.17 (IO13)
- net MOT_2.INDEX: now also U7.20 (IO16)
- net MOT_2.STEP: now also U7.18 (IO14)
- net RXD0: now also D2.3, R15.1; no longer J5.3 (Pin_3)
- net TXD0: now also D3.3, R16.2; no longer J5.2 (Pin_2)
- net USB_D+: now also R18.1, U7.24 (USB_D+); no longer R18.2
- net USB_D-: now also R17.1, U7.23 (USB_D-); no longer R17.2
- net VTX.RX: now reaches U7.11 (IO7)
- net VTX.TX: now reaches U7.12 (IO8)
- net MOT_1.~{EN}: now reaches U7.13 (IO9)
- net MOT_2.~{EN}: now reaches U7.16 (IO12)
- net TXD1: now reaches U7.21 (IO17)
- net TXD1: now also R20.2
- net MOT_1.UART: now reaches U7.22 (IO18)
- net MOT_1.UART: now also R20.1
- net IO21: now reaches U7.25 (IO21)
- net CTRL.RX: now reaches U7.29 (IO34)
- net CTRL.TX: now reaches U7.30 (IO48)
- net DIN: now reaches U7.31 (IO35)
- net DIN: now also D4.1 (DIN)
- net IO36: now reaches U7.32 (IO36)
- net +3.3V renamed +3V3
- net +3V3: now also D2.2, D3.2, L4.2; no longer J5.1 (Pin_1)
- new net: J5.3 (Pin_3), R16.1
- new net: D4.3 (DOUT), D5.1 (DIN)
- new net: J5.2 (Pin_2), R15.2
- new net: J5.1 (Pin_1), L4.1
- new net +5V: C35.1, C36.1, D4.2 (VDD), D5.2 (VDD)
- new net D+: R18.2
- new net D-: R17.2
- no-connect marks 0 -> 13
Other:
- moved on the sheet: J5, R17, R18

Commit message: Done, and completed bom
Parts:
- added TP10, TP11, TP12, TP13, TP14, TP15, TP16, TP17, TP18, TP19, TP21, TP22, TP23, TP6, TP7, TP8, TP9: TestPoint, TestPoint:TestPoint_Pad_D1.5mm, symbol Connector:TestPoint
- C34: renamed from C32; LCSC# (none) -> C14442
- C35: renamed from C33; LCSC# (none) -> C14442
- C36: renamed from C34; LCSC# (none) -> C14445
- C37: renamed from C35; LCSC# (none) -> C14442
- C38: renamed from C36; LCSC# (none) -> C14442
- J5: LCSC# (none) -> C7501262
- R16: renamed from R15; LCSC# (none) -> C105588
- R17: renamed from R16; LCSC# (none) -> C105588
- R18: renamed from R17; LCSC# (none) -> C2906858
- R19: renamed from R18; LCSC# (none) -> C2906858
- R20: renamed from R19; LCSC# (none) -> C2906861
- R21: renamed from R20; LCSC# (none) -> C2906864
- SW2: value EN -> B3U-1000P
- SW3: value BOOT -> B3U-1000P
- renumbered C31 to C33, L4 to L5
Connections:
- net CTRL.RX: now also TP11.1
- net CTRL.TX: now also TP10.1
- net IMU.SCL: now also TP6.1
- net IMU.SDA: now also TP7.1
- net MOT_1.DIAG: now also TP16.1
- net MOT_1.DIR: now also TP13.1
- net MOT_1.INDEX: now also TP17.1
- net MOT_1.STEP: now also TP12.1
- net MOT_1.UART: now also TP14.1
- net MOT_1.~{EN}: now also TP15.1
- net MOT_2.DIAG: now also TP22.1
- net MOT_2.DIR: now also TP19.1
- net MOT_2.INDEX: now also TP23.1
- net MOT_2.STEP: now also TP18.1
- net MOT_2.~{EN}: now also TP21.1
- net VTX.RX: now also TP9.1
- net VTX.TX: now also TP8.1

Commit message: Fixed Bom and added more GND fill
Parts:
- C34, C35, C37, C38: LCSC# C14442 -> C307331
- TP10, TP11, TP12, TP13, TP14, TP15, TP16, TP17, TP18, TP19, TP21, TP22, TP23, TP6, TP7, TP8, TP9: now left out of the parts list
Changed lines of the file:
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@@
 		(body_style 1)
 		(exclude_from_sim no)
-		(in_bom yes)
+		(in_bom no)
 		(on_board yes)
 		(in_pos_files yes)
@@
 		(body_style 1)
 		(exclude_from_sim no)
-		(in_bom yes)
+		(in_bom no)
 		(on_board yes)
 		(in_pos_files yes)
@@
 		(body_style 1)
 		(exclude_from_sim no)
-		(in_bom yes)
+		(in_bom no)
 		(on_board yes)
 		(in_pos_files yes)
@@
 			)
 		)
-		(property "LCSC#" "C14442"
+		(property "LCSC#" "C307331"
 			(at 147.32 43.18 0)
 			(hide yes)
@@
 		(body_style 1)
 		(exclude_from_sim no)
-		(in_bom yes)
+		(in_bom no)
 		(on_board yes)
 		(in_pos_files yes)
@@
 		(body_style 1)
 		(exclude_from_sim no)
-		(in_bom yes)
+		(in_bom no)
 		(on_board yes)
 		(in_pos_files yes)
@@
 		(body_style 1)
 		(exclude_from_sim no)
-		(in_bom yes)
+		(in_bom no)
 		(on_board yes)
 		(in_pos_files yes)
@@
 		(body_style 1)
 		(exclude_from_sim no)
-		(in_bom yes)
+		(in_bom no)
 		(on_board yes)
 		(in_pos_files yes)
@@
 		(body_style 1)
 		(exclude_from_sim no)
-		(in_bom yes)
+		(in_bom no)
 		(on_board yes)
 		(in_pos_files yes)
@@
 			)
 		)
-		(property "LCSC#" "C14442"
+		(property "LCSC#" "C307331"
 			(at 90.17 162.56 0)
 			(hide yes)
@@
 		(body_style 1)
 		(exclude_from_sim no)
-		(in_bom yes)
+		(in_bom no)
 		(on_board yes)
 		(in_pos_files yes)
@@
 		(body_style 1)
 		(exclude_from_sim no)
-		(in_bom yes)
+		(in_bom no)
 		(on_board yes)
 		(in_pos_files yes)
@@
 		(body_style 1)
 		(exclude_from_sim no)
-		(in_bom yes)
+		(in_bom no)
 		(on_board yes)
 		(in_pos_files yes)
@@
 		(body_style 1)
 		(exclude_from_sim no)
-		(in_bom yes)
+		(in_bom no)
 		(on_board yes)
 		(in_pos_files yes)
@@
 			)
 		)
-		(property "LCSC#" "C14442"
+		(property "LCSC#" "C307331"
 			(at 252.73 118.11 0)
 			(hide yes)
@@
 		(body_style 1)
 		(exclude_from_sim no)
-		(in_bom yes)
+		(in_bom no)
 		(on_board yes)
 		(in_pos_files yes)
@@
 		(body_style 1)
 		(exclude_from_sim no)
-		(in_bom yes)
+		(in_bom no)
 		(on_board yes)
 		(in_pos_files yes)
@@
 		(body_style 1)
 		(exclude_from_sim no)
-		(in_bom yes)
+		(in_bom no)
 		(on_board yes)
 		(in_pos_files yes)
@@
 			)
 		)
-		(property "LCSC#" "C14442"
+		(property "LCSC#" "C307331"
 			(at 125.73 162.56 0)
 			(hide yes)
@@
 		(body_style 1)
 		(exclude_from_sim no)
-		(in_bom yes)
+		(in_bom no)
 		(on_board yes)
 		(in_pos_files yes)
@@
 		(body_style 1)
 		(exclude_from_sim no)
-		(in_bom yes)
+		(in_bom no)
 		(on_board yes)
 		(in_pos_files yes)
