File: PCB/Balancing_cam/Power_in.kicad_sch (KiCad schematic)
At the start: 22 parts, among them J2 xt60

Commit message: Started with more stuff tho battery chargeis wip
Parts:
- removed BT1, BT2: Battery_Cell, symbol Device:Battery_Cell
- removed C10, C11, C12: C, symbol Device:C
- removed C13, C14: 22u, symbol Device:C
- removed C15: 1u, symbol Device:C
- removed C5: 22u, symbol Device:C_Polarized
- removed C6: 100n, symbol Device:C
- removed D2, D3: LED, symbol Device:LED
- removed J2: xt60, Connector_AMASS:AMASS_XT60-M_1x02_P7.20mm_Vertical, symbol Connector_Generic:Conn_01x02
- removed L1: L, symbol Device:L
- removed R10, R6, R7, R8, R9: R, symbol Device:R
- removed R11: 12k, symbol Device:R
- removed TH1: Thermistor_NTC, symbol Device:Thermistor_NTC
- removed U1: (no value), footprints:QFN-18 2mmx3mm, symbol symbols:MP2672A
- added J1: USB_C_Receptacle_USB2.0_16P, symbol Connector:USB_C_Receptacle_USB2.0_16P
- added R4, R5: 5.1k, symbol Device:R
Connections:
- net GND: now also J1.A1 (GND), J1.A12 (GND), J1.B1 (GND), J1.B12 (GND), J1.SH (SHIELD), R4.2, R5.2
- new net: J1.A5 (CC1), R4.1
- new net: J1.B5 (CC2), R5.1
- new net +5V: J1.A4 (VBUS), J1.A9 (VBUS), J1.B4 (VBUS), J1.B9 (VBUS)
- new net D+: J1.A6 (D+), J1.B6 (D+)
- new net D-: J1.A7 (D-), J1.B7 (D-)
- no-connect marks 0 -> 2
Other:
- title: (none) -> Balancing_cam

Commit message: Finalized schematic and pcb
Parts:
- added C19, C21, C24, C26, C45, C46: 100n, Capacitor_SMD:C_0402_1005Metric, symbol Device:C
- added C20, C25: 10u, Capacitor_SMD:C_0603_1608Metric, symbol Device:C
- added C22: 47u, Capacitor_SMD:C_0805_2012Metric, symbol Device:C
- added C23, C28: 33n, Capacitor_SMD:C_0402_1005Metric, symbol Device:C
- added C27: 100u, Capacitor_SMD:C_1206_3216Metric, symbol Device:C
- added D1: DSK24L, Diode_SMD:D_SOD-123F, symbol Device:D
- added F1, F2: Fuse, Fuse:Fuseholder_Littelfuse_Nano2_154x, symbol Device:Fuse
- added J1, J2: JST_PH, Connector_JST:JST_PH_S2B-PH-SM4-TB_1x02-1MP_P2.00mm_Horizontal, symbol Connector_Generic_MountingPin:Conn_01x02_MountingPin
- added J4: JST_XH, Connector_JST:JST_XH_B2B-XH-A_1x02_P2.50mm_Vertical, symbol Connector_Generic:Conn_01x02
- added L1, L2: 2u2, Inductor_SMD:L_1210_3225Metric, symbol Device:L
- added L14, L3: BLM18KG121TN1D, Inductor_SMD:L_0603_1608Metric, symbol Device:L
- added Q1: BC817, Package_TO_SOT_SMD:SOT-23, symbol Transistor_BJT:BC817
- added R25: 1k, Resistor_SMD:R_0402_1005Metric, symbol Device:R
- added R5: 52k3, Resistor_SMD:R_0402_1005Metric, symbol Device:R
- added R6, R9: 10k, Resistor_SMD:R_0402_1005Metric, symbol Device:R
- added R7: 14k7, Resistor_SMD:R_0402_1005Metric, symbol Device:R
- added R8: 30k9, Resistor_SMD:R_0402_1005Metric, symbol Device:R
- added SW1: SW_SPDT, footprints:SS12D10G5, symbol Switch:SW_SPDT
- added U3, U4: TPS62933, Package_TO_SOT_SMD:SOT-583-8, symbol Regulator_Switching:TPS62933
- added U5: USBLC6-2P6, Package_TO_SOT_SMD:SOT-666, symbol Power_Protection:USBLC6-2P6
- J3: renamed from J1; footprint (none) -> Connector_USB:USB_C_Receptacle_GCT_USB4105-xx-A_16P_TopMnt_Horizontal; LCSC# (none) -> C165948
- R10: renamed from R4; footprint (none) -> Resistor_SMD:R_0603_1608Metric
- R11: renamed from R5; footprint (none) -> Resistor_SMD:R_0603_1608Metric
Connections:
- net +5V: now also C22.1, C25.1, C26.1, C45.1, D1.1 (K), L1.2, L3.1, R5.2, U4.2 (EN), U4.3 (VIN), U5.5 (VBUS); no longer J3.A4 (VBUS), J3.A9 (VBUS), J3.B4 (VBUS), J3.B9 (VBUS)
- net D+: now also U5.4 (I/O2); no longer J3.A6 (D+), J3.B6 (D+)
- net D-: now also U5.6 (I/O1); no longer J3.A7 (D-), J3.B7 (D-)
- net GND: now also C20.2, C21.2, C22.2, C23.2, C25.2, C26.2, C27.2, C28.2, C45.2, C46.2, J1.MP (MountPin), J2.1 (Pin_2), J2.MP (MountPin), Q1.2 (E), R6.2, R7.2, R9.2, U3.4 (GND), U4.4 (GND), U5.2 (GND)
- new net: J4.1 (Pin_1), L3.2
- new net: J4.2 (Pin_2), L14.2
- new net: J1.1 (Pin_2), J2.2 (Pin_1)
- new net: R7.1, U3.1 (RT)
- new net: C19.2, L1.1, U3.5 (SW)
- new net: C19.1, U3.6 (BST)
- new net: C23.1, U3.7 (SS)
- new net: R5.1, R6.1, U3.8 (FB)
- new net: C28.1, U4.7 (SS)
- new net: C24.2, L2.1, U4.5 (SW)
- new net: C24.1, U4.6 (BST)
- new net: R8.1, R9.1, U4.8 (FB)
- new net: C46.1, Q1.1 (B), R25.2
- new net: L14.1, Q1.3 (C)
- new net: D1.2 (A), J3.A4 (VBUS), J3.A9 (VBUS), J3.B4 (VBUS), J3.B9 (VBUS)
- new net: J1.2 (Pin_1), SW1.2 (B)
- new net +3V3: C27.1, L2.2, R8.2
- new net DIRTY_D+: J3.A6 (D+), J3.B6 (D+), U5.3 (I/O2)
- new net DIRTY_D-: J3.A7 (D-), J3.B7 (D-), U5.1 (I/O1)
- new net FAN: R25.1
- new net VD: C20.1, C21.1, F2.2, U3.2 (EN), U3.3 (VIN)
- new net VS: F1.1, F2.1, SW1.3 (C)
- new net Vdrive: F1.2
- no-connect marks 2 -> 4
Other:
- moved on the sheet: J3, R10, R11

Commit message: Done, and completed bom
Parts:
- added TP1, TP2, TP3: TestPoint, TestPoint:TestPoint_Pad_D1.5mm, symbol Connector:TestPoint
- C19, C21, C24, C26: LCSC# (none) -> C14442
- C23, C28: LCSC# (none) -> C26404
- C29: renamed from C45; LCSC# (none) -> C14442
- C30: renamed from C46; LCSC# (none) -> C14442
- F1, F2: LCSC# C41371861 -> C108518
- J1, J2: footprint Connector_JST:JST_PH_S2B-PH-SM4-TB_1x02-1MP_P2.00mm_Horizontal -> footprints:JST_PH_S2B-PH-SM4-TB_1x02-1MP_P2.00mm_Horizontal
- L1: LCSC# (none) -> C3222669
- Q1: LCSC# (none) -> C52801
- R10, R11: LCSC# (none) -> C105580
- R12: renamed from R25; LCSC# (none) -> C2906864
- R5: LCSC# (none) -> C2998086
- R6, R9: LCSC# (none) -> C2906861
- R7: LCSC# (none) -> C2929988
- R8: LCSC# (none) -> C2933086
- renumbered L14 to L4
Connections:
- net +3V3: now also TP2.1
- net +5V: now also TP1.1
- net at L4.1, Q1.3 (C): now also TP3.1

Commit message: Fixed Bom and added more GND fill
Parts:
- C19, C21, C24, C26, C29, C30: LCSC# C14442 -> C307331
- C23, C28: LCSC# C26404 -> C472437
- TP1, TP2, TP3: now left out of the parts list
Changed lines of the file:
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@@
 		(body_style 1)
 		(exclude_from_sim no)
-		(in_bom yes)
+		(in_bom no)
 		(on_board yes)
 		(in_pos_files yes)
@@
 			)
 		)
-		(property "LCSC#" "C26404"
+		(property "LCSC#" "C472437"
 			(at 201.93 104.14 0)
 			(hide yes)
@@
 			)
 		)
-		(property "LCSC#" "C26404"
+		(property "LCSC#" "C472437"
 			(at 201.93 53.34 0)
 			(hide yes)
@@
 			)
 		)
-		(property "LCSC#" "C14442"
+		(property "LCSC#" "C307331"
 			(at 232.41 38.1 90)
 			(hide yes)
@@
 			)
 		)
-		(property "LCSC#" "C14442"
+		(property "LCSC#" "C307331"
 			(at 198.12 43.18 0)
 			(hide yes)
@@
 			)
 		)
-		(property "LCSC#" "C14442"
+		(property "LCSC#" "C307331"
 			(at 196.85 152.4 0)
 			(hide yes)
@@
 			)
 		)
-		(property "LCSC#" "C14442"
+		(property "LCSC#" "C307331"
 			(at 193.04 132.08 0)
 			(hide yes)
@@
 		(body_style 1)
 		(exclude_from_sim no)
-		(in_bom yes)
+		(in_bom no)
 		(on_board yes)
 		(in_pos_files yes)
@@
 			)
 		)
-		(property "LCSC#" "C14442"
+		(property "LCSC#" "C307331"
 			(at 232.41 88.9 90)
 			(hide yes)
@@
 		(body_style 1)
 		(exclude_from_sim no)
-		(in_bom yes)
+		(in_bom no)
 		(on_board yes)
 		(in_pos_files yes)
@@
 			)
 		)
-		(property "LCSC#" "C14442"
+		(property "LCSC#" "C307331"
 			(at 198.12 93.98 0)
 			(hide yes)
