File: PCB/Balancing_cam/_restore_backup_2026-08-08T16-02-50-453/IMU.kicad_sch (KiCad schematic)
At the start: 6 parts, among them U6 LSM6DS3

Commit message: Finalized schematic and pcb
Parts:
- removed C29, C30: 100n, Capacitor_SMD:C_0402_1005Metric, symbol Device:C
- removed R12, R13: 10k, Resistor_SMD:R_0402_1005Metric, symbol Device:R
- removed R14: 0R, Resistor_SMD:R_0402_1005Metric, symbol Device:R
- removed U6: LSM6DS3, Package_LGA:LGA-14_3x2.5mm_P0.5mm_LayoutBorder3x4y, symbol Sensor_Motion:LSM6DS3
- added C7: 100n, symbol Device:C
- added C8: 10n, symbol Device:C
- added C9: 2u2, symbol Device:C
- added IC1: ICM-42688-P, IIM42352, symbol SamacSys_Parts:ICM-42688-P
Connections:
- net +3V3: now also C7.1, C8.1, C9.1, IC1.5 (VDDIO), IC1.8 (VDD)
- net GND: now also C7.2, C8.2, C9.2, IC1.10 (RESV), IC1.11 (RESV), IC1.2 (RESV), IC1.3 (RESV), IC1.6 (GND), IC1.7 (RESV)
- net SCL: now also IC1.13 (SCL)
- net SDA: now also IC1.14 (SDA)
- new net +3.3V: IC1.12 (CS)
- new net INT: IC1.4 (INT)
- no-connect marks 4 -> 2
