File: PCB/Balancing_cam/_restore_backup_2026-08-08T16-02-50-453/Motor_drivers.kicad_sch (KiCad schematic)
At the start: 14 parts, among them U1 TMC2209-LA

Commit message: Finalized schematic and pcb
Parts:
- removed C8, C9: 100n, Capacitor_SMD:C_0402_1005Metric, symbol Device:C
- removed JP1, JP2: SolderJumper_2_Open, Jumper:SolderJumper-2_P1.3mm_Open_RoundedPad1.0x1.5mm, symbol Jumper:SolderJumper_2_Open
- added R12: 1k, symbol Device:R
- C52: renamed from C3; footprint Capacitor_SMD:C_0402_1005Metric -> Capacitor_SMD:C_0603_1608Metric
- C53: renamed from C4; footprint Capacitor_SMD:C_0402_1005Metric -> Capacitor_SMD:C_0603_1608Metric
- C54: renamed from C5; footprint Capacitor_SMD:CP_Elec_6.3x5.4 -> Capacitor_SMD:CP_Elec_10x10; LCSC# C2887272 -> (none)
- C55: renamed from C1; footprint Capacitor_SMD:C_0402_1005Metric -> Capacitor_SMD:C_0603_1608Metric
- C56: renamed from C2; footprint Capacitor_SMD:C_0402_1005Metric -> Capacitor_SMD:C_0603_1608Metric
- C73: renamed from C7; footprint Capacitor_SMD:C_0402_1005Metric -> Capacitor_SMD:C_0603_1608Metric
- U3: renamed from U1; LCSC# C2150710 -> (none)
- renumbered C6 to C69, R1 to R63, R2 to R68
Connections:
- net UART renamed RX
- net RX: now also R12.1
- net ~{EN} renamed EN
- new net TX: R12.2
Other:
- moved on the sheet: R63, R68
